File: Schematic/meteorito.sch (KiCad schematic (older format))
At the start: 12 parts, among them P1 DH22, P10 CONN_01X10, P2 GY-ML8511, P3 BMP180, P4 Hall, P5 Hall, P6 Hall, P7 CONN_01X10, P8 CONN_01X10, P9 CONN_01X10

Commit message: Corregir cambios
Parts:
- P1: footprint Pin_Headers:Pin_Header_Straight_1x03_Pitch2.54mm -> Resistor_THT:R_Axial_DIN0204_L3.6mm_D1.6mm_P5.08mm_Horizontal
- P10, P7, P8, P9: footprint (none) -> Connector_PinHeader_2.54mm:PinHeader_1x10_P2.54mm_Vertical
- P2: footprint Pin_Headers:Pin_Header_Straight_1x05_Pitch2.54mm -> Connector_PinHeader_2.54mm:PinHeader_1x05_P2.54mm_Vertical
- P3: footprint Pin_Headers:Pin_Header_Straight_1x04_Pitch2.54mm -> Connector_PinHeader_2.54mm:PinHeader_1x04_P2.54mm_Vertical
- P4, P5, P6: footprint (none) -> Connector_PinHeader_2.54mm:PinHeader_1x03_P2.54mm_Vertical
- R1: footprint (none) -> Resistor_THT:R_Axial_DIN0204_L3.6mm_D1.6mm_P2.54mm_Vertical
- R2: footprint (none) -> Resistor_THT:R_Axial_DIN0204_L3.6mm_D1.6mm_P7.62mm_Horizontal
Connections:
- net IO12 is gone; now on net IO27: P2.4 (P4)
- net +5V: now also P1.2 (P2); no longer P1.1 (P1)
- net IO16: now also P6.3 (P3)
- net IO17: now also P5.3 (P3)
- net IO23: now also P1.1 (P1); no longer P1.2 (P2)
- net IO0: no longer names the net of P7.7 (P7)
- net IO18: no longer names the net of P9.4 (P4)
- net IO19: no longer names the net of P9.5 (P5)
- net IO26: no longer names the net of P9.3 (P3)
- removed net SIG: P5.3 (P3), P6.3 (P3)
- no-connect marks 4 -> 29
Other:
- note added: "Sensor De Orientación \n"
- note added: "Sensor De Precipitación \n"
- note added: "\n\n"
- note removed: "Sensores Efecto Hall\n"
- moved on the sheet: P1
Changed lines of the file:
@@
 F 0 "P3" H 2370 2650 50  0000 C CNN
 F 1 "BMP180" V 2470 2400 50  0000 C CNN
-F 2 "Pin_Headers:Pin_Header_Straight_1x04_Pitch2.54mm" H 2370 2400 50  0001 C CNN
+F 2 "Connector_PinHeader_2.54mm:PinHeader_1x04_P2.54mm_Vertical" H 2370 2400 50  0001 C CNN
 F 3 "" H 2370 2400 50  0000 C CNN
 	1    2370 2400
@@
 F 0 "P2" H 2300 4175 50  0000 C CNN
 F 1 "GY-ML8511" V 2400 3875 50  0000 C CNN
-F 2 "Pin_Headers:Pin_Header_Straight_1x05_Pitch2.54mm" H 2300 3875 50  0001 C CNN
+F 2 "Connector_PinHeader_2.54mm:PinHeader_1x05_P2.54mm_Vertical" H 2300 3875 50  0001 C CNN
 F 3 "" H 2300 3875 50  0000 C CNN
 	1    2300 3875
@@
 $EndComp
 NoConn ~ 2100 3775
-$Comp
-L power:+5V #PWR04
-U 1 1 59FBB39C
-P 1860 945
-F 0 "#PWR04" H 1860 795 50  0001 C CNN
-F 1 "+5V" H 1860 1085 50  0000 C CNN
-F 2 "" H 1860 945 50  0000 C CNN
-F 3 "" H 1860 945 50  0000 C CNN
-	1    1860 945
-	1    0    0    -1
-$EndComp
 NoConn ~ 8135 2220
 NoConn ~ 8135 2120
@@
 L meteorito-rescue:CONN_01X03 P1
 U 1 1 5973B1A0
-P 2275 1095
-F 0 "P1" H 2275 1295 50  0000 C CNN
-F 1 "DH22" V 2375 1095 50  0000 C CNN
-F 2 "Pin_Headers:Pin_Header_Straight_1x03_Pitch2.54mm" H 2275 1095 50  0001 C CNN
-F 3 "" H 2275 1095 50  0000 C CNN
-	1    2275 1095
+P 2260 1025
+F 0 "P1" H 2260 1225 50  0000 C CNN
+F 1 "DH22" V 2360 1025 50  0000 C CNN
+F 2 "Resistor_THT:R_Axial_DIN0204_L3.6mm_D1.6mm_P5.08mm_Horizontal" H 2260 1025 50  0001 C CNN
+F 3 "" H 2260 1025 50  0000 C CNN
+	1    2260 1025
 	1    0    0    -1
 $EndComp
@@
 F 0 "R1" H 1930 6585 50  0000 L CNN
 F 1 "FOTORESISTENCIA" H 1930 6525 50  0000 L CNN
-F 2 "" H 1900 6565 50  0000 C CNN
+F 2 "Resistor_THT:R_Axial_DIN0204_L3.6mm_D1.6mm_P2.54mm_Vertical" H 1900 6565 50  0001 C CNN
 F 3 "" H 1900 6565 50  0000 C CNN
 	1    1900 6565
@@
 F 0 "R2" H 1930 6870 50  0000 L CNN
 F 1 "100" H 1930 6810 50  0000 L CNN
-F 2 "" H 1900 6850 50  0000 C CNN
+F 2 "Resistor_THT:R_Axial_DIN0204_L3.6mm_D1.6mm_P7.62mm_Horizontal" H 1900 6850 50  0001 C CNN
 F 3 "" H 1900 6850 50  0000 C CNN
 	1    1900 6850
@@
 F 0 "P8" H 7335 2810 50  0000 C CNN
 F 1 "CONN_01X10" V 7435 2260 50  0000 C CNN
-F 2 "" H 7335 2260 50  0000 C CNN
+F 2 "Connector_PinHeader_2.54mm:PinHeader_1x10_P2.54mm_Vertical" H 7335 2260 50  0001 C CNN
 F 3 "" H 7335 2260 50  0000 C CNN
 	1    7335 2260
@@
 F 0 "P7" H 6535 2815 50  0000 C CNN
 F 1 "CONN_01X10" V 6635 2265 50  0000 C CNN
-F 2 "" H 6535 2265 50  0000 C CNN
+F 2 "Connector_PinHeader_2.54mm:PinHeader_1x10_P2.54mm_Vertical" H 6535 2265 50  0001 C CNN
 F 3 "" H 6535 2265 50  0000 C CNN
 	1    6535 2265
@@
 F 0 "P9" H 7935 2820 50  0000 C CNN
 F 1 "CONN_01X10" V 8035 2270 50  0000 C CNN
-F 2 "" H 7935 2270 50  0000 C CNN
+F 2 "Connector_PinHeader_2.54mm:PinHeader_1x10_P2.54mm_Vertical" H 7935 2270 50  0001 C CNN
 F 3 "" H 7935 2270 50  0000 C CNN
 	1    7935 2270
@@
 F 0 "P10" H 8740 2835 50  0000 C CNN
 F 1 "CONN_01X10" V 8840 2285 50  0000 C CNN
-F 2 "" H 8740 2285 50  0000 C CNN
+F 2 "Connector_PinHeader_2.54mm:PinHeader_1x10_P2.54mm_Vertical" H 8740 2285 50  0001 C CNN
 F 3 "" H 8740 2285 50  0000 C CNN
 	1    8740 2285
@@
 Wire Wire Line
 	1900 6950 1900 7050
-Wire Notes Line
-	4305 5460 11220 5460
 Wire Notes Line
 	11220 4260 11220 4250
@@
 F 0 "P5" H 5300 4950 50  0000 C CNN
 F 1 "Hall" V 5400 4750 50  0000 C CNN
-F 2 "" H 5300 4750 50  0000 C CNN
+F 2 "Connector_PinHeader_2.54mm:PinHeader_1x03_P2.54mm_Vertical" H 5300 4750 50  0001 C CNN
 F 3 "" H 5300 4750 50  0000 C CNN
 	1    5300 4750
@@
 F 0 "P6" H 6500 4950 50  0000 C CNN
 F 1 "Hall" V 6600 4750 50  0000 C CNN
-F 2 "" H 6500 4750 50  0000 C CNN
+F 2 "Connector_PinHeader_2.54mm:PinHeader_1x03_P2.54mm_Vertical" H 6500 4750 50  0001 C CNN
 F 3 "" H 6500 4750 50  0000 C CNN
 	1    6500 4750
@@
 $EndComp
 Text Notes 5300 4200 0    50   ~ 0
-Sensores Efecto Hall\n
+\n\n
 Wire Notes Line
 	7150 4050 7150 5450
@@
 F 0 "P4" H 2200 5400 50  0000 C CNN
 F 1 "Hall" V 2300 5200 50  0000 C CNN
-F 2 "" H 2200 5200 50  0000 C CNN
+F 2 "Connector_PinHeader_2.54mm:PinHeader_1x03_P2.54mm_Vertical" H 2200 5200 50  0001 C CNN
 F 3 "" H 2200 5200 50  0000 C CNN
 	1    2200 5200
@@
 	6335 2315 6065 2315
 Wire Wire Line
-	6335 2415 6065 2415
-Wire Wire Line
 	6335 2515 6085 2515
 Wire Wire Line
@@
 Wire Wire Line
 	5940 4750 5940 4655
-Wire Wire Line
-	2075 1095 1860 1095
 Text Label 6065 1815 0    50   ~ 0
 GND
@@
 Text Label 6065 2315 0    50   ~ 0
 IO4
-Text Label 6065 2415 0    50   ~ 0
-IO0
 Text Label 6085 2515 0    50   ~ 0
 IO2
@@
 Text Label 9300 2735 2    50   ~ 0
 CMD
-Text Label 1860 1095 0    50   ~ 0
-IO23
 Text Label 4905 4850 0    50   ~ 0
-SIG
-Text Label 6105 4850 0    50   ~ 0
-SIG
-Wire Wire Line
-	2075 995  1860 995
-Wire Wire Line
-	1860 995  1860 945
+IO17
+Text Label 6070 4850 0    50   ~ 0
+IO16
+Wire Wire Line
+	2060 925  1845 925
 Wire Wire Line
 	2170 2450 2010 2450
@@
 Wire Wire Line
 	2170 2550 2010 2550
-Wire Wire Line
-	2100 3975 1980 3975
-Text Label 1980 3975 0    50   ~ 0
-IO12
+Text Label 2085 3975 2    50   ~ 0
+IO27
 Wire Wire Line
 	1750 5000 1750 5200
@@
 Wire Wire Line
 	1900 6710 1900 6665
-Wire Wire Line
-	1900 6465 1900 6370
 $Comp
 L power:GND #PWR0101
 U 1 1 5BAA240F
-P 1855 1220
-F 0 "#PWR0101" H 1855 970 50  0001 C CNN
-F 1 "GND" H 1860 1047 50  0000 C CNN
-F 2 "" H 1855 1220 50  0001 C CNN
-F 3 "" H 1855 1220 50  0001 C CNN
-	1    1855 1220
-	1    0    0    -1
-$EndComp
-Wire Wire Line
-	1855 1220 1855 1195
-Wire Wire Line
-	1855 1195 2075 1195
-Wire Wire Line
-	6335 1915 6065 1915
+P 1840 1150
+F 0 "#PWR0101" H 1840 900 50  0001 C CNN
+F 1 "GND" H 1845 977 50  0000 C CNN
+F 2 "" H 1840 1150 50  0001 C CNN
+F 3 "" H 1840 1150 50  0001 C CNN
+	1    1840 1150
+	1    0    0    -1
+$EndComp
+Wire Wire Line
+	1840 1150 1840 1125
+Wire Wire Line
+	1840 1125 2060 1125
 Wire Wire Line
 	7135 1910 6900 1910
 Wire Wire Line
 	7135 2010 6900 2010
-Wire Wire Line
-	8135 2120 8465 2120
-Wire Wire Line
-	8135 2220 8465 2220
-Text Label 8465 2120 2    50   ~ 0
-IO18
-Text Label 8465 2220 2    50   ~ 0
-IO19
-Wire Wire Line
-	8135 2020 8465 2020
-Text Label 8465 2020 2    50   ~ 0
-IO26
 Text Label 6910 2110 0    50   ~ 0
 IO21
@@
 Text Label 2175 6710 0    50   ~ 0
 IO13
+$Comp
+L power:+5V #PWR0102
+U 1 1 5BB55C40
+P 1695 970
+F 0 "#PWR0102" H 1695 820 50  0001 C CNN
+F 1 "+5V" H 1695 1110 50  0000 C CNN
+F 2 "" H 1695 970 50  0000 C CNN
+F 3 "" H 1695 970 50  0000 C CNN
+	1    1695 970
+	1    0    0    -1
+$EndComp
+Text Label 1845 925  0    50   ~ 0
+IO23
+Wire Wire Line
+	2060 1025 1695 1025
+Wire Wire Line
+	1695 1025 1695 970
+Wire Notes Line
+	5650 4065 5650 5460
+Wire Notes Line
+	4305 5460 11220 5460
+Text Notes 4605 4210 0    50   ~ 0
+Sensor De Precipitación \n
+Text Notes 5945 4205 0    50   ~ 0
+Sensor De Orientación \n
+NoConn ~ 6335 2115
+NoConn ~ 6335 2215
+NoConn ~ 6335 2315
+NoConn ~ 6335 2415
+NoConn ~ 6335 2515
+NoConn ~ 6335 2615
+NoConn ~ 6335 2715
+NoConn ~ 7135 2510
+NoConn ~ 7135 2610
+NoConn ~ 7135 2710
+NoConn ~ 7135 1810
+NoConn ~ 7135 1910
+NoConn ~ 8135 1820
+NoConn ~ 8135 1920
+NoConn ~ 8135 2420
+NoConn ~ 8135 2520
+NoConn ~ 8135 2620
+NoConn ~ 8135 2720
+NoConn ~ 8940 2035
+NoConn ~ 8940 2135
+NoConn ~ 8940 2235
+NoConn ~ 8940 2335
+NoConn ~ 8940 2435
+NoConn ~ 8940 2635
+NoConn ~ 8940 2735
+Wire Wire Line
+	1900 6370 1900 6465
+Wire Wire Line
+	2100 3975 2085 3975
+Wire Wire Line
+	6335 1915 6065 1915
 $EndSCHEMATC

Commit message: Corrección
Se colocaron la tierra y el VCC y se volvio a rootear lo faltante
Connections:
- net 3.3V is gone; now on net +3V3: P9.8 (P8)
- net TCK is gone; now on net IO13: P9.9 (P9)
- net VCC is gone; now on net +5V: P8.8 (P8)
- no-connect marks 29 -> 26
Changed lines of the file:
@@
 	7135 2310 6910 2310
 Wire Wire Line
-	7135 2410 6915 2410
-Wire Wire Line
-	7135 2510 6915 2510
-Wire Wire Line
 	8135 2320 8475 2320
 Wire Wire Line
 	8135 2720 8440 2720
-Wire Wire Line
-	8135 2520 8460 2520
 Wire Wire Line
 	8135 2420 8470 2420
@@
 $EndComp
 Wire Wire Line
-	6335 1815 6065 1815
-Wire Wire Line
 	8940 2735 9300 2735
 Wire Wire Line
@@
 Wire Wire Line
 	8940 1935 9280 1935
-Wire Wire Line
-	8940 1835 9280 1835
 $Comp
 L power:GND #PWR09
@@
 Wire Wire Line
 	5940 4750 5940 4655
-Text Label 6065 1815 0    50   ~ 0
-GND
 Text Label 6065 1915 0    50   ~ 0
 IO27
@@
 Text Label 6910 2310 0    50   ~ 0
 IO16
-Text Label 6915 2410 0    50   ~ 0
-GND
-Text Label 6915 2510 0    50   ~ 0
-VCC
 Text Label 6930 2610 0    50   ~ 0
 TD0
@@
 Text Label 8470 2420 2    50   ~ 0
 IO5
-Text Label 8460 2520 2    50   ~ 0
-3.3V
-Text Label 8440 2620 2    50   ~ 0
-TCK
 Text Label 8440 2720 2    50   ~ 0
 SD3
-Text Label 9280 1835 2    50   ~ 0
-GND
 Text Label 9280 1935 2    50   ~ 0
 NC
@@
 NoConn ~ 6335 2615
 NoConn ~ 6335 2715
-NoConn ~ 7135 2510
 NoConn ~ 7135 2610
 NoConn ~ 7135 2710
@@
 NoConn ~ 8135 1920
 NoConn ~ 8135 2420
-NoConn ~ 8135 2520
-NoConn ~ 8135 2620
 NoConn ~ 8135 2720
 NoConn ~ 8940 2035
@@
 Wire Wire Line
 	6335 1915 6065 1915
+$Comp
+L power:GND #PWR0103
+U 1 1 5BEA53DD
+P 9410 1855
+F 0 "#PWR0103" H 9410 1605 50  0001 C CNN
+F 1 "GND" H 9415 1682 50  0000 C CNN
+F 2 "" H 9410 1855 50  0001 C CNN
+F 3 "" H 9410 1855 50  0001 C CNN
+	1    9410 1855
+	1    0    0    -1
+$EndComp
+$Comp
+L power:GND #PWR0104
+U 1 1 5BEA5417
+P 5920 1855
+F 0 "#PWR0104" H 5920 1605 50  0001 C CNN
+F 1 "GND" H 5925 1682 50  0000 C CNN
+F 2 "" H 5920 1855 50  0001 C CNN
+F 3 "" H 5920 1855 50  0001 C CNN
+	1    5920 1855
+	1    0    0    -1
+$EndComp
+Wire Wire Line
+	5920 1855 5920 1815
+Wire Wire Line
+	5920 1815 6335 1815
+Wire Wire Line
+	9410 1855 9410 1835
+Wire Wire Line
+	8940 1835 9410 1835
+$Comp
+L power:GND #PWR0105
+U 1 1 5BEAA495
+P 6795 2435
+F 0 "#PWR0105" H 6795 2185 50  0001 C CNN
+F 1 "GND" H 6800 2262 50  0000 C CNN
+F 2 "" H 6795 2435 50  0001 C CNN
+F 3 "" H 6795 2435 50  0001 C CNN
+	1    6795 2435
+	1    0    0    -1
+$EndComp
+Wire Wire Line
+	6795 2435 6795 2410
+Wire Wire Line
+	6795 2410 7135 2410
+$Comp
+L power:+5V #PWR0106
+U 1 1 5BEACE6C
+P 6830 1700
+F 0 "#PWR0106" H 6830 1550 50  0001 C CNN
+F 1 "+5V" H 6845 1873 50  0000 C CNN
+F 2 "" H 6830 1700 50  0001 C CNN
+F 3 "" H 6830 1700 50  0001 C CNN
+	1    6830 1700
+	1    0    0    -1
+$EndComp
+Wire Wire Line
+	6830 2510 7135 2510
+Wire Wire Line
+	6830 2510 6830 1700
+$Comp
+L power:+3.3V #PWR0107
+U 1 1 5BEB4B8C
+P 8535 1690
+F 0 "#PWR0107" H 8535 1540 50  0001 C CNN
+F 1 "+3.3V" H 8550 1863 50  0000 C CNN
+F 2 "" H 8535 1690 50  0001 C CNN
+F 3 "" H 8535 1690 50  0001 C CNN
+	1    8535 1690
+	1    0    0    -1
+$EndComp
+Wire Wire Line
+	8535 2520 8535 1690
+Wire Wire Line
+	8135 2520 8535 2520
+Text Label 8440 2620 2    50   ~ 0
+IO13
 $EndSCHEMATC

Commit message: Remove NC pins
Connections:
- net NC: no longer names the net of P10.2 (P2)
- net NC: no longer P10.8 (P8)
- no-connect marks 26 -> 28
Changed lines of the file:
@@
 	8940 2635 9300 2635
 Wire Wire Line
-	8940 2535 9300 2535
-Wire Wire Line
 	8940 2435 9300 2435
 Wire Wire Line
@@
 Wire Wire Line
 	8940 2035 9280 2035
-Wire Wire Line
-	8940 1935 9280 1935
 $Comp
 L power:GND #PWR09
@@
 Text Label 8440 2720 2    50   ~ 0
 SD3
-Text Label 9280 1935 2    50   ~ 0
-NC
 Text Label 9280 2035 2    50   ~ 0
 SVN
@@
 Text Label 9300 2435 2    50   ~ 0
 TMS
-Text Label 9300 2535 2    50   ~ 0
-NC
 Text Label 9300 2635 2    50   ~ 0
 SD2
@@
 Text Label 8440 2620 2    50   ~ 0
 IO13
+NoConn ~ 8940 1935
+NoConn ~ 8940 2535
 $EndSCHEMATC

Commit message: Rerouted
Parts:
- P1: footprint Resistor_THT:R_Axial_DIN0204_L3.6mm_D1.6mm_P5.08mm_Horizontal -> Connector_PinHeader_2.54mm:PinHeader_1x03_P2.54mm_Vertical
Connections:
- net +3V3: now also P2.2 (P2), P2.5 (P5)
- net +5V: no longer P2.1 (P1), P2.5 (P5)
- net IO13: no longer R1.2, R2.1
- net IO16: now also P5.3 (P3); no longer P6.3 (P3)
- net IO17: now also P6.3 (P3); no longer P5.3 (P3)
- net IO27: no longer P2.4 (P4)
- net IO33: now also P2.4 (P4)
- net IO35: now also R1.2, R2.1
Changed lines of the file:
@@
 	1    0    0    -1
 $EndComp
-$Comp
-L power:+5V #PWR010
-U 1 1 59FBB879
-P 1960 3675
-F 0 "#PWR010" H 1960 3525 50  0001 C CNN
-F 1 "+5V" H 1960 3815 50  0000 C CNN
-F 2 "" H 1960 3675 50  0000 C CNN
-F 3 "" H 1960 3675 50  0000 C CNN
-	1    1960 3675
-	1    0    0    -1
-$EndComp
-NoConn ~ 2100 3775
 NoConn ~ 8135 2220
 NoConn ~ 8135 2120
@@
 F 0 "P1" H 2260 1225 50  0000 C CNN
 F 1 "DH22" V 2360 1025 50  0000 C CNN
-F 2 "Resistor_THT:R_Axial_DIN0204_L3.6mm_D1.6mm_P5.08mm_Horizontal" H 2260 1025 50  0001 C CNN
+F 2 "Connector_PinHeader_2.54mm:PinHeader_1x03_P2.54mm_Vertical" H 2260 1025 50  0001 C CNN
 F 3 "" H 2260 1025 50  0000 C CNN
 	1    2260 1025
@@
 	1875 2350 2170 2350
 Wire Wire Line
-	2100 3675 1960 3675
-Wire Wire Line
 	1875 2350 1875 2355
 Wire Wire Line
@@
 L power:GND #PWR09
 U 1 1 5BA50CA8
-P 1910 3930
-F 0 "#PWR09" H 1910 3680 50  0001 C CNN
-F 1 "GND" H 1915 3757 50  0000 C CNN
-F 2 "" H 1910 3930 50  0001 C CNN
-F 3 "" H 1910 3930 50  0001 C CNN
-	1    1910 3930
-	1    0    0    -1
-$EndComp
-Wire Wire Line
-	1910 3930 1910 3875
-Wire Wire Line
-	1910 3875 2100 3875
-$Comp
-L power:+5V #PWR01
-U 1 1 5BA55AD4
-P 1695 4055
-F 0 "#PWR01" H 1695 3905 50  0001 C CNN
-F 1 "+5V" H 1710 4228 50  0000 C CNN
-F 2 "" H 1695 4055 50  0001 C CNN
-F 3 "" H 1695 4055 50  0001 C CNN
-	1    1695 4055
-	1    0    0    -1
-$EndComp
-Wire Wire Line
-	2100 4075 2045 4075
-Wire Wire Line
-	2045 4075 2045 4180
-Wire Wire Line
-	2045 4180 1695 4180
-Wire Wire Line
-	1695 4180 1695 4055
+P 1690 3915
+F 0 "#PWR09" H 1690 3665 50  0001 C CNN
+F 1 "GND" H 1695 3742 50  0000 C CNN
+F 2 "" H 1690 3915 50  0001 C CNN
+F 3 "" H 1690 3915 50  0001 C CNN
+	1    1690 3915
+	1    0    0    -1
+$EndComp
 Wire Wire Line
 	2000 5100 1985 5100
@@
 CMD
 Text Label 4905 4850 0    50   ~ 0
+IO16
+Text Label 6070 4850 0    50   ~ 0
 IO17
-Text Label 6070 4850 0    50   ~ 0
-IO16
 Wire Wire Line
 	2060 925  1845 925
@@
 	2170 2550 2010 2550
 Text Label 2085 3975 2    50   ~ 0
-IO27
+IO33
 Wire Wire Line
 	1750 5000 1750 5200
@@
 IO23
 Text Label 2175 6710 0    50   ~ 0
-IO13
+IO35
 $Comp
 L power:+5V #PWR0102
@@
 NoConn ~ 8940 1935
 NoConn ~ 8940 2535
+$Comp
+L power:+3.3V #PWR0108
+U 1 1 5C9D397E
+P 1500 3985
+F 0 "#PWR0108" H 1500 3835 50  0001 C CNN
+F 1 "+3.3V" H 1515 4158 50  0000 C CNN
+F 2 "" H 1500 3985 50  0001 C CNN
+F 3 "" H 1500 3985 50  0001 C CNN
+	1    1500 3985
+	1    0    0    -1
+$EndComp
+$Comp
+L power:+3.3V #PWR0109
+U 1 1 5C9D39DE
+P 1865 3735
+F 0 "#PWR0109" H 1865 3585 50  0001 C CNN
+F 1 "+3.3V" H 1880 3908 50  0000 C CNN
+F 2 "" H 1865 3735 50  0001 C CNN
+F 3 "" H 1865 3735 50  0001 C CNN
+	1    1865 3735
+	1    0    0    -1
+$EndComp
+Wire Wire Line
+	2100 3775 1865 3775
+Wire Wire Line
+	1865 3775 1865 3735
+NoConn ~ 2100 3675
+Wire Wire Line
+	1690 3875 1690 3915
+Wire Wire Line
+	1690 3875 2100 3875
+Wire Wire Line
+	1885 4075 1885 4160
+Wire Wire Line
+	1885 4160 1500 4160
+Wire Wire Line
+	1500 4160 1500 3985
+Wire Wire Line
+	2100 4075 1885 4075
 $EndSCHEMATC
