File: Schematic/meteorito.kicad_pcb (KiCad board)
At the start: 2 copper layers, 95.3 x 89.4 mm, 19 parts, among them P1 DH22, P10 CONN_01X10, P2 GY-ML8511, P3 BMP180, P4 Hall, P5 Hall, P6 Hall, P7 CONN_01X10, P8 CONN_01X10, P9 CONN_01X10

Commit message: Add hole M3
Parts:
- added REF**: MountingHole_3.2mm_M3_ISO14580_Pad, Mounting_Holes:MountingHole_3.2mm_M3_ISO14580_Pad, F.Cu at (47.2, 63.0)
- added REF**: MountingHole_3.2mm_M3_ISO14580_Pad, Mounting_Holes:MountingHole_3.2mm_M3_ISO14580_Pad, F.Cu at (124.2, 60.5)
- added REF**: MountingHole_3.2mm_M3_ISO14580_Pad, Mounting_Holes:MountingHole_3.2mm_M3_ISO14580_Pad, F.Cu at (45.9, 137.8)
- added REF**: MountingHole_3.2mm_M3_ISO14580_Pad, Mounting_Holes:MountingHole_3.2mm_M3_ISO14580_Pad, F.Cu at (127.5, 137.5)
- moved REF*** 6.81 mm to (124.5, 72.7)
- moved G*** 5.20 mm to (130.3, 85.5)
Changed lines of the file:
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@@
     (tracks 144)
     (zones 0)
-    (modules 19)
+    (modules 23)
     (nets 40)
   )
@@
     (43 Eco2.User user)
     (44 Edge.Cuts user)
-    (45 Margin user hide)
+    (45 Margin user)
     (46 B.CrtYd user)
     (47 F.CrtYd user)
@@
     (visible_elements 7FFFFFFF)
     (pcbplotparams
-      (layerselection 0x00030_80000001)
-      (usegerberextensions false)
+      (layerselection 0x010f0_ffffffff)
+      (usegerberextensions true)
       (usegerberattributes false)
       (usegerberadvancedattributes false)
@@
       (outputformat 1)
       (mirror false)
-      (drillshape 1)
+      (drillshape 0)
       (scaleselection 1)
-      (outputdirectory ""))
+      (outputdirectory "gerbers_meteorito_v01/"))
   )
   (net 0 "")
@@
   )
   (module LOGO (layer B.Cu)
-    (at 126.1618 82.30616 270)
+    (at 130.3 85.45 270)
     (fp_text reference G*** (at 0 0 270) (layer B.SilkS) hide
       (effects (font (size 1.524 1.524) (thickness 0.3)) (justify mirror))
@@
   )
   (module Symbols:OSHW-Logo_11.4x12mm_SilkScreen (layer F.Cu)
-    (at 122.25 66.25 90)
+    (at 124.45 72.7 90)
     (descr "Open Source Hardware Logo")
     (tags "Logo OSHW")
@@
     )
   )
+  (module Mounting_Holes:MountingHole_3.2mm_M3_ISO14580_Pad (layer F.Cu)
+    (at 47.2 63.05)
+    (descr "Mounting Hole 3.2mm, M3, ISO14580")
+    (tags "mounting hole 3.2mm m3 iso14580")
+    (attr virtual)
+    (fp_text reference REF** (at 0 -3.75) (layer F.SilkS)
+      (effects (font (size 1 1) (thickness 0.15)))
+    )
+    (fp_text value MountingHole_3.2mm_M3_ISO14580_Pad (at 0 3.75) (layer F.Fab)
+      (effects (font (size 1 1) (thickness 0.15)))
+    )
+    (fp_text user %R (at 0.3 0) (layer F.Fab)
+      (effects (font (size 1 1) (thickness 0.15)))
+    )
+    (fp_circle (center 0 0) (end 2.75 0) (layer Cmts.User) (width 0.15))
+    (fp_circle (center 0 0) (end 3 0) (layer F.CrtYd) (width 0.05))
+    (pad 1 thru_hole circle (at 0 0) (size 5.5 5.5) (drill 3.2) (layers *.Cu *.Mask))
+  )
+  (module Mounting_Holes:MountingHole_3.2mm_M3_ISO14580_Pad (layer F.Cu)
+    (at 124.2 60.55)
+    (descr "Mounting Hole 3.2mm, M3, ISO14580")
+    (tags "mounting hole 3.2mm m3 iso14580")
+    (attr virtual)
+    (fp_text reference REF** (at 0 -3.75) (layer F.SilkS)
+      (effects (font (size 1 1) (thickness 0.15)))
+    )
+    (fp_text value MountingHole_3.2mm_M3_ISO14580_Pad (at 0 3.75) (layer F.Fab)
+      (effects (font (size 1 1) (thickness 0.15)))
+    )
+    (fp_text user %R (at 0.3 0) (layer F.Fab)
+      (effects (font (size 1 1) (thickness 0.15)))
+    )
+    (fp_circle (center 0 0) (end 2.75 0) (layer Cmts.User) (width 0.15))
+    (fp_circle (center 0 0) (end 3 0) (layer F.CrtYd) (width 0.05))
+    (pad 1 thru_hole circle (at 0 0) (size 5.5 5.5) (drill 3.2) (layers *.Cu *.Mask))
+  )
+  (module Mounting_Holes:MountingHole_3.2mm_M3_ISO14580_Pad (layer F.Cu)
+    (at 45.9 137.8)
+    (descr "Mounting Hole 3.2mm, M3, ISO14580")
+    (tags "mounting hole 3.2mm m3 iso14580")
+    (attr virtual)
+    (fp_text reference REF** (at 0 -3.75) (layer F.SilkS)
+      (effects (font (size 1 1) (thickness 0.15)))
+    )
+    (fp_text value MountingHole_3.2mm_M3_ISO14580_Pad (at 0 3.75) (layer F.Fab)
+      (effects (font (size 1 1) (thickness 0.15)))
+    )
+    (fp_text user %R (at 0.3 0) (layer F.Fab)
+      (effects (font (size 1 1) (thickness 0.15)))
+    )
+    (fp_circle (center 0 0) (end 2.75 0) (layer Cmts.User) (width 0.15))
+    (fp_circle (center 0 0) (end 3 0) (layer F.CrtYd) (width 0.05))
+    (pad 1 thru_hole circle (at 0 0) (size 5.5 5.5) (drill 3.2) (layers *.Cu *.Mask))
+  )
+  (module Mounting_Holes:MountingHole_3.2mm_M3_ISO14580_Pad (layer F.Cu)
+    (at 127.55 137.5)
+    (descr "Mounting Hole 3.2mm, M3, ISO14580")
+    (tags "mounting hole 3.2mm m3 iso14580")
+    (attr virtual)
+    (fp_text reference REF** (at 0 -3.75) (layer F.SilkS)
+      (effects (font (size 1 1) (thickness 0.15)))
+    )
+    (fp_text value MountingHole_3.2mm_M3_ISO14580_Pad (at 0 3.75) (layer F.Fab)
+      (effects (font (size 1 1) (thickness 0.15)))
+    )
+    (fp_text user %R (at 0.3 0) (layer F.Fab)
+      (effects (font (size 1 1) (thickness 0.15)))
+    )
+    (fp_circle (center 0 0) (end 2.75 0) (layer Cmts.User) (width 0.15))
+    (fp_circle (center 0 0) (end 3 0) (layer F.CrtYd) (width 0.05))
+    (pad 1 thru_hole circle (at 0 0) (size 5.5 5.5) (drill 3.2) (layers *.Cu *.Mask))
+  )
   (gr_text v0.1 (at 66.65 96.6 90) (layer F.SilkS)
     (effects (font (size 1.5 1.5) (thickness 0.3)))
@@
     (effects (font (size 2.5 2.5) (thickness 0.3)) (justify mirror))
   )
-  (gr_text "Con apoyo de:" (at 120.4722 74.38136 90) (layer B.SilkS)
+  (gr_text "Con apoyo de:" (at 124.05 78.85 90) (layer B.SilkS)
     (effects (font (size 2.5 2.5) (thickness 0.3)) (justify mirror))
   )
@@
     (connect_pads (clearance 0.508))
     (min_thickness 0.254)
-    (fill yes (arc_segments 16) (thermal_gap 0.508) (thermal_bridge_width 0.508))
+    (fill (arc_segments 16) (thermal_gap 0.508) (thermal_bridge_width 0.508))
     (polygon
       (pts
@@
     (connect_pads (clearance 0.508))
     (min_thickness 0.254)
-    (fill yes (arc_segments 16) (thermal_gap 0.508) (thermal_bridge_width 0.508))
+    (fill (arc_segments 16) (thermal_gap 0.508) (thermal_bridge_width 0.508))
     (polygon
       (pts

Commit message: Screw Hole
Parts:
- removed the REF** at (47.2, 63.0)
- removed the REF** at (124.2, 60.5)
- removed the REF** at (127.5, 137.5)
- added REF**: MountingHole_3.2mm_M3_ISO14580_Pad, Mounting_Holes:MountingHole_3.2mm_M3_ISO14580_Pad, F.Cu at (48.4, 64.7)
- added REF**: MountingHole_3.2mm_M3_ISO14580_Pad, Mounting_Holes:MountingHole_3.2mm_M3_ISO14580_Pad, F.Cu at (126.0, 64.5)
- added REF**: MountingHole_3.2mm_M3_ISO14580_Pad, Mounting_Holes:MountingHole_3.2mm_M3_ISO14580_Pad, F.Cu at (126.1, 136.1)
- moved REF** 3.05 mm to (48.6, 136.3)
- moved G*** 2.58 mm to (130.8, 88.0)
